File: GB_DMG_PSU.kicad_pcb (KiCad board)
At the start: 2 copper layers, 15 x 65 mm, 21 parts, among them J2 Conn_01x04, U1 R1283K001C-TR

Commit message: final touches
Parts:
- added C8: 4,7µF, Capacitor_SMD:C_0603_1608Metric, F.Cu at (107.8, 73.8)
- C6: value C -> 47pF
- R1: value R -> 10k
- R2: value R -> 42k
- R3, R6: value R -> 1k
- R4: value R -> 6,8k
- R5: value R -> 100k
- moved C5 4.35 mm to (108.2, 69.3), turned to 0 degrees
- moved R1 3.28 mm to (105.3, 69.2), turned to 180 degrees
- moved R2 1.84 mm to (105.2, 72.2), turned to 0 degrees
- moved R3 1.61 mm to (105.2, 70.8), turned to 0 degrees
- moved C1 0.45 mm to (107.8, 76.2)
- moved C4 0.07 mm to (107.8, 77.7)
Routing:
- net FB1: track 9.02 -> 13.0 mm
- net Net-(C5-Pad1): track 1.38 -> 2.39 mm
- net GND: vias 11 -> 10
Other:
- board text added: "-18V"
- board text added: "5V"
- board text added: "GND"
- board text added: "VCC"

Commit message: manufacturing files
Parts:
- C10, C7: value C -> as large as possible
Changed lines of the file:
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@@
 			(outputformat 1)
 			(mirror no)
-			(drillshape 1)
+			(drillshape 0)
 			(scaleselection 1)
-			(outputdirectory "")
+			(outputdirectory "gerber")
 		)
 	)
@@
 			)
 		)
-		(property "Value" "C"
+		(property "Value" "as large as possible"
 			(at 0 2.35 90)
 			(layer "F.Fab")
@@
 			)
 		)
-		(property "Value" "C"
+		(property "Value" "as large as possible"
 			(at 0 2.35 270)
 			(layer "F.Fab")

Commit message: don't need backups online
Parts:
- C6: value 47pF -> 330pF
Changed lines of the file:
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@@
 			)
 		)
-		(property "Value" "47pF"
+		(property "Value" "330pF"
 			(at 0 1.43 90)
 			(layer "F.Fab")

Commit message: V2
Parts:
- removed C5: 68pF, Capacitor_SMD:C_0603_1608Metric
- removed C6: 330pF, Capacitor_SMD:C_0603_1608Metric
- removed C7: as large as possible, Capacitor_Tantalum_SMD:CP_EIA-3528-12_Kemet-T
- removed C8: 4,7µF, Capacitor_SMD:C_0603_1608Metric
- removed L1, L2: 4,7µH, Inductor_SMD:L_0805_2012Metric
- removed R2: 42k, Resistor_SMD:R_0603_1608Metric
- removed U1: R1283K001C-TR, footprints:PE-DFNPL2730-12-180404_NMD
- added C11: 10µF, Capacitor_SMD:C_0603_1608Metric, F.Cu at (73.2, 85.0)
- added C12: 10µF, Capacitor_SMD:C_0603_1608Metric, F.Cu at (72.4, 62.2)
- added C13: 1µF, Capacitor_SMD:C_0603_1608Metric, F.Cu at (81.2, 61.5)
- added C14: 10µF, Capacitor_SMD:C_0603_1608Metric, F.Cu at (78.9, 58.5)
- added C15: 1µF, Capacitor_SMD:C_0603_1608Metric, F.Cu at (81.2, 66.5)
- added C16: 10uF, Capacitor_SMD:C_0603_1608Metric, F.Cu at (78.0, 53.1)
- added C18: 100nF, Capacitor_SMD:C_0603_1608Metric, F.Cu at (78.0, 47.1)
- added C9: 1µF, Capacitor_SMD:C_0603_1608Metric, F.Cu at (75.8, 85.8)
- added D4: D, Diode_SMD:D_SOD-323, F.Cu at (79.0, 60.0)
- added D5: D, Diode_SMD:D_SOD-323, F.Cu at (81.3, 63.2)
- added D6: D, Diode_SMD:D_SOD-323, F.Cu at (82.0, 59.2)
- added D7: 18V, Diode_SMD:D_SOD-323, F.Cu at (82.0, 72.8)
- added F1: Fuse, Fuse:Fuse_1206_3216Metric, F.Cu at (81.2, 36.0)
- added J3: Conn_01x02, Connector_JST:JST_PH_S2B-PH-K_1x02_P2.00mm_Horizontal, B.Cu at (81.8, 52.5)
- added J4: Conn_01x01, Connector_PinHeader_2.54mm:PinHeader_1x01_P2.54mm_Vertical, F.Cu at (70.8, 38.0)
- added JP1: Jumper, Jumper:SolderJumper-2_P1.3mm_Open_RoundedPad1.0x1.5mm, F.Cu at (71.5, 45.5)
- added L3: 10µH, Inductor_SMD:L_APV_ANR5040, F.Cu at (79.5, 86.8)
- added L4: 10µH, Inductor_SMD:L_APV_ANR5040, F.Cu at (79.5, 80.8)
- added L5: 10µH, Inductor_SMD:L_APV_ANR5040, F.Cu at (76.8, 64.2)
- added Q1: BSS84, Package_TO_SOT_SMD:SOT-23, F.Cu at (81.5, 44.8)
- added R10: 100k, Resistor_SMD:R_0603_1608Metric, F.Cu at (71.6, 56.8)
- added R11: 100k, Resistor_SMD:R_0603_1608Metric, F.Cu at (75.1, 55.2)
- added R12: 6,8k, Resistor_SMD:R_0603_1608Metric, F.Cu at (75.1, 56.8)
- added R13: 15k, Resistor_SMD:R_0603_1608Metric, F.Cu at (81.2, 65.0)
- added R14: TBD, Resistor_SMD:R_0603_1608Metric, F.Cu at (80.2, 72.8)
- added R7: 100k, Resistor_SMD:R_0603_1608Metric, F.Cu at (74.2, 78.2)
- added R8: 100k, Resistor_SMD:R_0603_1608Metric, F.Cu at (72.5, 72.5)
- added R9: 100k, Resistor_SMD:R_0603_1608Metric, F.Cu at (71.6, 55.3)
- added U2: LGS6302B5, Package_TO_SOT_SMD:SOT-23-5, F.Cu at (73.3, 59.5)
- added U3: LGS6302B5, Package_TO_SOT_SMD:SOT-23-5, F.Cu at (74.5, 82.2)
- added U4: MCP73831, Package_TO_SOT_SMD:SOT-23-5, F.Cu at (78.0, 50.0)
- C1: value 4,7µF -> 10µF
- C3: footprint Capacitor_SMD:C_0603_1608Metric -> Capacitor_SMD:C_1206_3216Metric
- C4: value 100nF -> 10µF
- D2: value D -> LED_CHR; footprint Diode_SMD:D_SOD-323 -> LED_THT:LED_D3.0mm
- R1: value 10k -> 33k
- R3: value 1k -> 100k
- R4: value 6,8k -> 1K
- R5: value 100k -> 100K
- R6: value 1k -> 2K
- moved C3 45.5 mm to (79.8, 38.2)
- moved R6 44.9 mm to (78.0, 45.6), turned to 0 degrees
- moved R4 41.9 mm to (74.0, 52.8), turned to -90 degrees
- moved R5 39.7 mm to (81.5, 47.5), turned to 180 degrees
- moved D3 38.6 mm to (74.2, 45.0), turned to 90 degrees
- moved D2 37.0 mm to (72.2, 50.5), turned to 90 degrees
- moved C1 36.1 mm to (73.2, 86.5)
- moved R3 32.9 mm to (72.5, 74.0)
- moved R1 32.7 mm to (74.2, 79.8), turned to 0 degrees
- moved C4 30.4 mm to (77.5, 75.8), turned to 180 degrees
- moved C10 28.5 mm to (74.5, 38.0), turned to 180 degrees
- moved J2 26.3 mm to (73.2, 34.8)
- moved C2 23.3 mm to (77.5, 77.2), turned to 180 degrees
- moved D1 18.3 mm to (80.8, 76.8), turned to 0 degrees
Connections:
- C3 pad 1: -VDC -> -18V
- C4 pad 1: VREF -> +5V
- D1 pad 2: /buck+ -> /sw2
- D2 pad 1: /buck- -> Net-(D2-K)
- D2 pad 2: -VDC -> VIN
- D3 pad 1: Net-(D3-K) -> VCC
- D3 pad 2: VCC -> VIN
- J2 pad 2: -VDC -> -18V
- J2 pad 4: Net-(D3-K) -> Net-(J2-Pin_4)
- R1 pad 1: FB1 -> Net-(U3-FB)
- R3 pad 1: +5V -> Net-(U3-EN)
- R3 pad 2: Net-(C5-Pad1) -> GND
- R4 pad 1: FB2 -> Net-(D2-K)
- R4 pad 2: VREF -> Net-(U4-STAT)
- R5 pad 1: -VDC -> GND
- R5 pad 2: FB2 -> VIN
- R6 pad 1: -VDC -> GND
Routing:
- net -VDC: track 68.6 -> 0.00 mm
- net VCC: track 21.7 -> 77.5 mm, vias 5 -> 7
- net -18V: track 0.00 -> 48.8 mm
- net Net-(D3-K): track 45.0 -> 0.00 mm
- net VIN: track 0.00 -> 28.5 mm, vias 0 -> 2
- net VBAT: track 0.00 -> 13.9 mm
- net FB1: track 13.0 -> 0.00 mm
- net Net-(J2-Pin_4): track 0.00 -> 12.7 mm
- net Net-(U3-EN): track 0.00 -> 10.4 mm
- net /sw2: track 0.00 -> 9.49 mm, vias 0 -> 2
- net FB2: track 6.82 -> 0.00 mm
- net +18V: track 0.00 -> 5.91 mm
- net VREF: track 5.27 -> 0.00 mm
- net /pump2: track 0.00 -> 5.02 mm
- net Net-(U4-STAT): track 0.00 -> 4.65 mm, vias 0 -> 2
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- added copper zone on F.Cu, net +18V
- added copper zone on F.Cu, net /pump1
- added copper zone on F.Cu, net /pump2
- added copper zone on F.Cu, net /sw
- added copper zone on F.Cu, net /sw2
- added copper zone on F.Cu, net /sw3
- removed copper zone on F.Cu, net -VDC
- removed copper zone on F.Cu, net /buck+
- removed copper zone on F.Cu, net /buck-
Other:
- board text added: "+ -"
- board text added: "chg"

Commit message: some things i missed
Parts:
- removed F1: Fuse, Fuse:Fuse_1206_3216Metric
- added J1: Conn_01x01, Connector_PinHeader_2.54mm:PinHeader_1x01_P2.54mm_Vertical, F.Cu at (70.8, 34.8)
- added JP2: Jumper, Jumper:SolderJumper-2_P1.3mm_Open_RoundedPad1.0x1.5mm, F.Cu at (82.5, 50.5)
- added RV1: Varistor, Resistor_SMD:R_0603_1608Metric, F.Cu at (71.5, 43.2)
- C1, C11, C12, C14, C16, C2, C4: footprint Capacitor_SMD:C_0603_1608Metric -> Capacitor_SMD:C_0805_2012Metric
- C10: footprint Capacitor_Tantalum_SMD:CP_EIA-3528-12_Kemet-T -> Capacitor_SMD:C_1206_3216Metric
- C3: footprint Capacitor_SMD:C_1206_3216Metric -> Capacitor_SMD:C_0805_2012Metric
- moved J3 2.64 mm to (82.6, 55.0)
- moved C3 1.41 mm to (80.8, 37.2)
- moved C10 1.25 mm to (75.5, 37.2), turned to 0 degrees
- moved C4 0.75 mm to (77.5, 75.0)
- moved J4 0.75 mm to (70.8, 37.2)
- moved R4 0.71 mm to (74.5, 52.2), turned to 0 degrees
- moved C1 0.50 mm to (73.3, 87.0)
- moved C14 0.42 mm to (79.0, 58.1)
- moved C2 0.25 mm to (77.5, 77.0)
- moved D2 0.25 mm to (72.2, 50.3)
- moved C16 0.15 mm to (78.2, 53.1)
Connections:
- D3 pad 1: VCC -> Net-(D3-K)
- J2 pad 4: Net-(J2-Pin_4) -> VCC
- J3 pad 1: GND -> VBAT
- J3 pad 2: VBAT -> GND
- Q1 pad 2: VCC -> Net-(D3-K)
Routing:
- net Net-(D3-K): track 0.00 -> 27.1 mm, vias 0 -> 2
- net Net-(J2-Pin_4): track 12.7 -> 0.00 mm
- net Net-(U4-STAT): track 4.65 -> 2.23 mm, vias 2 -> 0
- net VCC: track 77.5 -> 79.9 mm, vias 7 -> 6
- net VBAT: track 13.9 -> 16.1 mm
- net +5V: track 56.6 -> 58.4 mm
- net GND: track 0.00 -> 0.78 mm, vias 22 -> 32
- net -18V: track 48.8 -> 49.5 mm
Other:
- board text added: "batt+"

Commit message: final tweaks before manufacture
Parts:
- added C5: 1µF, Capacitor_SMD:C_0603_1608Metric, F.Cu at (78.8, 72.5)
- C10: value as large as possible -> 100µF
- C18: value 100nF -> 1µF
- C3: value 10µF -> 100µF; footprint Capacitor_SMD:C_0805_2012Metric -> Capacitor_SMD:C_1206_3216Metric
- R4: value 1K -> 2K
- moved C3 0.35 mm to (81.1, 37.2)
- moved D7 0.23 mm to (82.0, 72.5)
- moved R14 0.23 mm to (80.3, 72.5)
Routing:
- net -18V: track 49.5 -> 50.9 mm
Other:
- board text added: "-18"
- board text removed: "-18V"
