File: GB_DMG_PSU.kicad_pcb (KiCad board)
At the start: 2 copper layers, 15 x 65 mm, 32 parts, among them J2 Conn_01x04, U2 LGS6302B5, U3 LGS6302B5

Commit message: moved some vias
Parts:
- moved R10 0.37 mm to (72.0, 56.8)
- moved R9 0.37 mm to (72.0, 55.3)
Routing:
- net GND: vias 72 -> 75
Changed lines of the file:
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@@
 	(footprint "Resistor_SMD:R_0603_1608Metric"
 		(layer "F.Cu")
-		(at 71.633348 55.345826)
+		(at 72 55.345826)
 		(descr "Resistor SMD 0603 (1608 Metric), square (rectangular) end terminal, IPC-7351 nominal, (Body size source: IPC-SM-782 page 72, https://www.pcb-3d.com/wordpress/wp-content/uploads/ipc-sm-782a_amendment_1_and_2.pdf), generated with kicad-footprint-generator")
 		(tags "resistor")
@@
 	(footprint "Resistor_SMD:R_0603_1608Metric"
 		(layer "F.Cu")
-		(at 71.633348 56.845826)
+		(at 72 56.845826)
 		(descr "Resistor SMD 0603 (1608 Metric), square (rectangular) end terminal, IPC-7351 nominal, (Body size source: IPC-SM-782 page 72, https://www.pcb-3d.com/wordpress/wp-content/uploads/ipc-sm-782a_amendment_1_and_2.pdf), generated with kicad-footprint-generator")
 		(tags "resistor")
@@
 	)
 	(via
+		(at 70.25 51.5)
+		(size 0.7)
+		(drill 0.3)
+		(layers "F.Cu" "B.Cu")
+		(free yes)
+		(net 1)
+	)
+	(via
 		(at 70.25 86.5)
 		(size 0.7)
@@
 	)
 	(via
-		(at 73.25 57.5)
+		(at 73.25 57.75)
 		(size 0.7)
 		(drill 0.3)
@@
 	)
 	(via
-		(at 72.5 75.5)
+		(at 70.25 49.75)
 		(size 0.7)
 		(drill 0.3)
@@
 	)
 	(via
-		(at 77 90)
+		(at 72.5 75.5)
 		(size 0.7)
 		(drill 0.3)
@@
 	)
 	(via
-		(at 83.75 48)
+		(at 77 90)
 		(size 0.7)
 		(drill 0.3)
@@
 	)
 	(via
+		(at 70.25 56.75)
+		(size 0.7)
+		(drill 0.3)
+		(layers "F.Cu" "B.Cu")
+		(free yes)
+		(net 1)
+	)
+	(via
 		(at 70.25 65.5)
 		(size 0.7)
@@
 	)
 	(via
+		(at 70.25 55)
+		(size 0.7)
+		(drill 0.3)
+		(layers "F.Cu" "B.Cu")
+		(free yes)
+		(net 1)
+	)
+	(via
 		(at 78 56.9)
 		(size 0.7)
@@
 	)
 	(via
-		(at 70.25 67.25)
+		(at 70.25 53.25)
 		(size 0.7)
 		(drill 0.3)
@@
 	)
 	(via
-		(at 70.25 62)
+		(at 70.25 67.25)
 		(size 0.7)
 		(drill 0.3)
@@
 	)
 	(via
-		(at 73.366652 61)
+		(at 70.25 62)
 		(size 0.7)
 		(drill 0.3)
@@
 	)
 	(via
-		(at 83.75 56.75)
+		(at 73.366652 61)
 		(size 0.7)
 		(drill 0.3)
@@
 	)
 	(via
-		(at 83.75 65.5)
+		(at 83.75 56.75)
 		(size 0.7)
 		(drill 0.3)
@@
 	)
 	(via
-		(at 83.75 46.25)
+		(at 83.75 65.5)
 		(size 0.7)
 		(drill 0.3)
@@
 	(segment
 		(start 72.25 54.25)
-		(end 72.5 54.5)
+		(end 72.825 54.825)
 		(width 0.2)
 		(layer "F.Cu")
@@
 	)
 	(segment
-		(start 72.5 54.5)
-		(end 72.5 55.304174)
+		(start 72.825 54.825)
+		(end 72.825 55.345826)
 		(width 0.2)
 		(layer "F.Cu")
@@
 	)
 	(segment
-		(start 72.5 55.304174)
-		(end 72.458348 55.345826)
-		(width 0.2)
-		(layer "F.Cu")
-		(net 6)
-	)
-	(segment
 		(start 73.325 71.075)
 		(end 73.325 72.25)
@@
 	)
 	(segment
-		(start 70.808348 56.845826)
-		(end 70.808348 57.191696)
+		(start 71.175 56.845826)
+		(end 71.175 57.558348)
 		(width 0.2)
 		(layer "F.Cu")
@@
 	)
 	(segment
-		(start 70.75 55.404174)
-		(end 70.75 56.787478)
+		(start 71.116652 55.404174)
+		(end 71.116652 56.787478)
 		(width 0.2)
 		(layer "F.Cu")
@@
 	)
 	(segment
-		(start 70.808348 57.191696)
+		(start 71.175 57.558348)
 		(end 72.116652 58.5)
 		(width 0.2)
@@
 		(width 0.2)
 		(layer "F.Cu")
-		(net 7)
-	)
-	(segment
-		(start 70.75 56.787478)
-		(end 70.808348 56.845826)
-		(width 0.2)
-		(layer "F.Cu")

Commit message: BOM/gerbers
Parts:
- C3: value 100µF -> 22µF
Other:
- board text added: "DMG-PSU V1,1"
Changed lines of the file:
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@@
 			)
 		)
-		(property "Value" "100µF"
+		(property "Value" "22µF"
 			(at 0 1.85 0)
 			(layer "F.Fab")
@@
 		)
 	)
-	(gr_text "CERN-OHL-P"
-		(at 77 50.577587 -0)
+	(gr_text "DMG-PSU V1,1"
+		(at 77 51 0)
 		(layer "F.SilkS")
 		(effects
@@
 				(bold yes)
 			)
+			(justify bottom)
 		)
 	)
@@
 		)
 	)
+	(gr_text "CERN-OHL-P"
+		(at 77 38.5 0)
+		(layer "B.SilkS")
+		(effects
+			(font
+				(size 1 1)
+				(thickness 0.2)
+				(bold yes)
+			)
+			(justify mirror)
+		)
+	)
 	(gr_text "-18"
 		(at 71 32.25 -0)
@@
 	)
 	(segment
-		(start 70.85 29.59)
-		(end 73.25 27.19)
+		(start 71.75 63.6)
+		(end 71.75 67.75)
 		(width 0.5)
 		(layer "B.Cu")
@@
 	)
 	(segment
-		(start 71.75 63.6)
-		(end 71.75 67.75)
+		(start 71 29.44)
+		(end 73.25 27.19)
 		(width 0.5)
 		(layer "B.Cu")
@@
 	)
 	(segment
-		(start 71.75 54.25)
-		(end 71.75 53.25)
+		(start 71.75 53.25)
+		(end 71 52.5)
 		(width 0.5)
 		(layer "B.Cu")
@@
 	)
 	(segment
-		(start 70.85 52.35)
-		(end 70.85 29.59)
+		(start 73.25 76)
+		(end 73.25 71)
 		(width 0.5)
 		(layer "B.Cu")
@@
 	)
 	(segment
-		(start 73.25 76)
-		(end 73.25 71)
+		(start 71.75 54.25)
+		(end 71.75 53.25)
 		(width 0.5)
 		(layer "B.Cu")
@@
 	)
 	(segment
-		(start 71.75 53.25)
-		(end 70.85 52.35)
+		(start 71 52.5)
+		(end 71 29.44)
 		(width 0.5)
 		(layer "B.Cu")
