File: GB_DMG_PSU.kicad_sch (KiCad schematic)
At the start: 21 parts, among them J2 Conn_01x04, U1 R1283K001C-TR

Commit message: final touches
Parts:
- added C8: 4,7µF, Capacitor_SMD:C_0603_1608Metric, symbol Device:C_Small
- C6: value C -> 47pF
- R1: value R -> 10k
- R2: value R -> 42k
- R3, R6: value R -> 1k
- R4: value R -> 6,8k
- R5: value R -> 100k
Connections:
- net GND: now also C8.2
- net VCC: now also C8.1
Changed lines of the file:
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@@
 	)
 	(junction
+		(at 106.68 43.18)
+		(diameter 0)
+		(color 0 0 0 0)
+	)
+	(junction
 		(at 109.22 66.04)
 		(diameter 0)
@@
 	)
 	(junction
+		(at 99.06 43.18)
+		(diameter 0)
+		(color 0 0 0 0)
+	)
+	(junction
 		(at 66.04 78.74)
 		(diameter 0)
@@
 	(wire
 		(pts
-			(xy 106.68 39.37) (xy 106.68 38.1)
+			(xy 99.06 43.18) (xy 100.33 43.18)
+		)
+		(stroke
+			(width 0)
+			(type default)
+		)
+	)
+	(wire
+		(pts
+			(xy 106.68 46.99) (xy 106.68 43.18)
 		)
 		(stroke
@@
 	(wire
 		(pts
+			(xy 106.68 43.18) (xy 106.68 38.1)
+		)
+		(stroke
+			(width 0)
+			(type default)
+		)
+	)
+	(wire
+		(pts
 			(xy 105.41 73.66) (xy 109.22 73.66)
 		)
@@
 	(wire
 		(pts
+			(xy 105.41 43.18) (xy 106.68 43.18)
+		)
+		(stroke
+			(width 0)
+			(type default)
+		)
+	)
+	(wire
+		(pts
 			(xy 105.41 73.66) (xy 105.41 74.93)
 		)
@@
 	(wire
 		(pts
+			(xy 99.06 43.18) (xy 99.06 45.72)
+		)
+		(stroke
+			(width 0)
+			(type default)
+		)
+	)
+	(wire
+		(pts
 			(xy 85.09 86.36) (xy 85.09 87.63)
 		)
@@
 	(wire
 		(pts
-			(xy 99.06 38.1) (xy 99.06 45.72)
+			(xy 99.06 38.1) (xy 99.06 43.18)
 		)
 		(stroke
@@
 		(dnp no)
 		(property "Reference" "R2"
-			(at 61.214 67.31 0)
+			(at 60.198 67.31 0)
 			(effects
 				(font
@@
 			)
 		)
-		(property "Value" "R"
-			(at 61.214 69.85 0)
+		(property "Value" "42k"
+			(at 60.198 69.85 0)
 			(effects
 				(font
@@
 			)
 		)
-		(property "Value" "C"
+		(property "Value" "47pF"
 			(at 85.09 76.2062 0)
 			(effects
@@
 			)
 		)
-		(property "Value" "R"
+		(property "Value" "10k"
 			(at 70.866 85.09 0)
 			(effects
@@
 		(lib_name "GND_1")
 		(lib_id "power:GND")
-		(at 106.68 39.37 0)
+		(at 106.68 46.99 0)
 		(unit 1)
 		(exclude_from_sim no)
@@
 		(dnp no)
 		(property "Reference" "#PWR02"
-			(at 106.68 45.72 0)
+			(at 106.68 53.34 0)
 			(effects
 				(font
@@
 		)
 		(property "Value" "GND"
-			(at 106.68 43.18 0)
+			(at 106.68 50.8 0)
 			(effects
 				(font
@@
 		)
 		(property "Footprint" ""
-			(at 106.68 39.37 0)
+			(at 106.68 46.99 0)
 			(effects
 				(font
@@
 		)
 		(property "Datasheet" ""
-			(at 106.68 39.37 0)
+			(at 106.68 46.99 0)
 			(effects
 				(font
@@
 		)
 		(property "Description" "Power symbol creates a global label with name \"GND\" , ground"
-			(at 106.68 39.37 0)
+			(at 106.68 46.99 0)
 			(effects
 				(font
@@
 			)
 		)
-		(property "Value" "R"
+		(property "Value" "1k"
 			(at 68.326 69.85 0)
 			(effects
@@
 			)
 		)
-		(property "Value" "R"
+		(property "Value" "6,8k"
 			(at 86.106 85.09 0)
 			(effects
@@
 		(dnp no)
 		(property "Reference" "R5"
-			(at 76.454 67.31 0)
+			(at 74.168 67.31 0)
 			(effects
 				(font
@@
 			)
 		)
-		(property "Value" "R"
-			(at 76.454 69.85 0)
+		(property "Value" "100k"
+			(at 74.168 69.85 0)
 			(effects
 				(font
@@
 	)
 	(symbol
+		(lib_id "Device:C_Small")
+		(at 102.87 43.18 90)
+		(unit 1)
+		(exclude_from_sim no)
+		(in_bom yes)
+		(on_board yes)
+		(dnp no)
+		(property "Reference" "C8"
+			(at 112.776 44.196 90)
+			(effects
+				(font
+					(size 1.27 1.27)
+				)
+				(justify left)
+			)
+		)
+		(property "Value" "4,7µF"
+			(at 112.776 41.656 90)
+			(effects
+				(font
+					(size 1.27 1.27)
+				)
+				(justify left)
+			)
+		)
+		(property "Footprint" "Capacitor_SMD:C_0603_1608Metric"
+			(at 102.87 43.18 0)
+			(effects
+				(font
+					(size 1.27 1.27)
+				)
+				(hide yes)
+			)
+		)
+		(property "Datasheet" "~"
+			(at 102.87 43.18 0)
+			(effects
+				(font
+					(size 1.27 1.27)
+				)
+				(hide yes)
+			)
+		)
+		(property "Description" "Unpolarized capacitor, small symbol"
+			(at 102.87 43.18 0)
+			(effects
+				(font
+					(size 1.27 1.27)
+				)
+				(hide yes)
+			)
+		)
+		(pin "1"
+		)
+		(pin "2"
+		)
+		(instances
+			(project "GB_DMG_PSU"
+				(path "/3b465854-de6d-4c79-a332-83f1753a534a"
+					(reference "C8")
+					(unit 1)
+				)
+			)
+		)
+	)
+	(symbol
 		(lib_name "GND_1")
 		(lib_id "power:GND")
@@
 			)
 		)
-		(property "Value" "R"
+		(property "Value" "1k"
 			(at 83.566 69.85 0)
 			(effects

Commit message: manufacturing files
Parts:
- C10, C7: value C -> as large as possible
- C6: value 47pF -> 330pF
Other:
- moved on the sheet: C3, C4
Changed lines of the file:
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@@
 	(wire
 		(pts
-			(xy 134.62 66.04) (xy 134.62 67.31)
+			(xy 140.97 66.04) (xy 140.97 67.31)
 		)
 		(stroke
@@
 	(wire
 		(pts
-			(xy 124.46 72.39) (xy 124.46 73.66)
+			(xy 130.81 72.39) (xy 130.81 73.66)
 		)
 		(stroke
@@
 	(wire
 		(pts
-			(xy 124.46 66.04) (xy 124.46 67.31)
+			(xy 130.81 66.04) (xy 130.81 67.31)
 		)
 		(stroke
@@
 	(wire
 		(pts
-			(xy 134.62 72.39) (xy 134.62 73.66)
+			(xy 140.97 72.39) (xy 140.97 73.66)
 		)
 		(stroke
@@
 	(global_label "VREF"
 		(shape input)
-		(at 134.62 66.04 90)
+		(at 140.97 66.04 90)
 		(fields_autoplaced yes)
 		(effects
@@
 		)
 		(property "Intersheetrefs" "${INTERSHEET_REFS}"
-			(at 134.62 58.4586 90)
+			(at 140.97 58.4586 90)
 			(effects
 				(font
@@
 		(lib_name "GND_1")
 		(lib_id "power:GND")
-		(at 124.46 73.66 0)
+		(at 130.81 73.66 0)
 		(unit 1)
 		(exclude_from_sim no)
@@
 		(dnp no)
 		(property "Reference" "#PWR016"
-			(at 124.46 80.01 0)
+			(at 130.81 80.01 0)
 			(effects
 				(font
@@
 		)
 		(property "Value" "GND"
-			(at 124.46 77.47 0)
+			(at 130.81 77.47 0)
 			(effects
 				(font
@@
 		)
 		(property "Footprint" ""
-			(at 124.46 73.66 0)
+			(at 130.81 73.66 0)
 			(effects
 				(font
@@
 		)
 		(property "Datasheet" ""
-			(at 124.46 73.66 0)
+			(at 130.81 73.66 0)
 			(effects
 				(font
@@
 		)
 		(property "Description" "Power symbol creates a global label with name \"GND\" , ground"
-			(at 124.46 73.66 0)
+			(at 130.81 73.66 0)
 			(effects
 				(font
@@
 			)
 		)
-		(property "Value" "47pF"
+		(property "Value" "330pF"
 			(at 85.09 76.2062 0)
 			(effects
@@
 		(on_board yes)
 		(dnp no)
-		(fields_autoplaced yes)
 		(property "Reference" "C7"
 			(at 115.57 68.0338 0)
@@
 			)
 		)
-		(property "Value" "C"
-			(at 115.57 70.5738 0)
+		(property "Value" "as large as possible"
+			(at 107.442 75.692 0)
 			(effects
 				(font
@@
 		(lib_name "GND_1")
 		(lib_id "power:GND")
-		(at 134.62 73.66 0)
+		(at 140.97 73.66 0)
 		(unit 1)
 		(exclude_from_sim no)
@@
 		(dnp no)
 		(property "Reference" "#PWR018"
-			(at 134.62 80.01 0)
+			(at 140.97 80.01 0)
 			(effects
 				(font
@@
 		)
 		(property "Value" "GND"
-			(at 134.62 77.47 0)
+			(at 140.97 77.47 0)
 			(effects
 				(font
@@
 		)
 		(property "Footprint" ""
-			(at 134.62 73.66 0)
+			(at 140.97 73.66 0)
 			(effects
 				(font
@@
 		)
 		(property "Datasheet" ""
-			(at 134.62 73.66 0)
+			(at 140.97 73.66 0)
 			(effects
 				(font
@@
 		)
 		(property "Description" "Power symbol creates a global label with name \"GND\" , ground"
-			(at 134.62 73.66 0)
+			(at 140.97 73.66 0)
 			(effects
 				(font
@@
 	(symbol
 		(lib_id "Device:C_Small")
-		(at 134.62 69.85 0)
+		(at 140.97 69.85 0)
 		(unit 1)
 		(exclude_from_sim no)
@@
 		(dnp no)
 		(property "Reference" "C4"
-			(at 137.16 68.5862 0)
+			(at 143.51 68.5862 0)
 			(effects
 				(font
@@
 		)
 		(property "Value" "100nF"
-			(at 137.16 71.1262 0)
+			(at 143.51 71.1262 0)
 			(effects
 				(font
@@
 		)
 		(property "Footprint" "Capacitor_SMD:C_0603_1608Metric"
-			(at 134.62 69.85 0)
+			(at 140.97 69.85 0)
 			(effects
 				(font
@@
 		)
 		(property "Datasheet" "~"
-			(at 134.62 69.85 0)
+			(at 140.97 69.85 0)
 			(effects
 				(font
@@
 		)
 		(property "Description" "Unpolarized capacitor, small symbol"
-			(at 134.62 69.85 0)
+			(at 140.97 69.85 0)
 			(effects
 				(font
@@
 	(symbol
 		(lib_id "power:-VDC")
-		(at 124.46 66.04 0)
+		(at 130.81 66.04 0)
 		(unit 1)
 		(exclude_from_sim no)
@@
 		(dnp no)
 		(property "Reference" "#PWR012"
-			(at 124.46 68.58 0)
+			(at 130.81 68.58 0)
 			(effects
 				(font
@@
 		)
 		(property "Value" "-VDC"
-			(at 125.73 65.532 0)
+			(at 132.08 65.532 0)
 			(effects
 				(font
@@
 		)
 		(property "Footprint" ""
-			(at 124.46 66.04 0)
+			(at 130.81 66.04 0)
 			(effects
 				(font
@@
 		)
 		(property "Datasheet" ""
-			(at 124.46 66.04 0)
+			(at 130.81 66.04 0)
 			(effects
 				(font
@@
 		)
 		(property "Description" "Power symbol creates a global label with name \"-VDC\""
-			(at 124.46 66.04 0)
+			(at 130.81 66.04 0)
 			(effects
 				(font
@@
 	(symbol
 		(lib_id "Device:C_Small")
-		(at 124.46 69.85 0)
+		(at 130.81 69.85 0)
 		(unit 1)
 		(exclude_from_sim no)
@@
 		(dnp no)
 		(property "Reference" "C3"
-			(at 127 68.5862 0)
+			(at 133.35 68.5862 0)
 			(effects
 				(font
@@
 		)
 		(property "Value" "10µF"
-			(at 127 71.1262 0)
+			(at 133.35 71.1262 0)
 			(effects
 				(font
@@
 		)
 		(property "Footprint" "Capacitor_SMD:C_0603_1608Metric"
-			(at 124.46 69.85 0)
+			(at 130.81 69.85 0)
 			(effects
 				(font
@@
 		)
 		(property "Datasheet" "~"
-			(at 124.46 69.85 0)
+			(at 130.81 69.85 0)
 			(effects
 				(font
@@
 		)
 		(property "Description" "Unpolarized capacitor, small symbol"
-			(at 124.46 69.85 0)
+			(at 130.81 69.85 0)
 			(effects
 				(font
@@
 		(dnp no)
 		(property "Reference" "C10"
-			(at 107.188 62.484 0)
+			(at 107.188 61.976 0)
 			(effects
 				(font
@@
 			)
 		)
-		(property "Value" "C"
-			(at 107.188 65.024 0)
+		(property "Value" "as large as possible"
+			(at 107.188 64.516 0)
 			(effects
 				(font

Commit message: more changes
Parts:
- removed D3: D, Diode_SMD:D_SOD-323, symbol Device:D_Small
- added C16: 10uF, Capacitor_SMD:C_0603_1608Metric, symbol Device:C_Small
- added C18: 100nF, Capacitor_SMD:C_0402_1005Metric, symbol Device:C_Small
- added C9: TBD, Capacitor_SMD:C_0402_1005Metric, symbol Device:C_Small
- added D4: LED_CHR, LED_SMD:LED_0402_1005Metric, symbol Device:LED_Small
- added D5: D_Schottky_Small, Diode_SMD:D_SOD-323, symbol Device:D_Schottky_Small
- added J1, J3: Conn_01x02, symbol Connector_Generic:Conn_01x02
- added Q1: BSS84, Package_TO_SOT_SMD:SOT-23, symbol Transistor_FET:BSS84
- added R7: 2K, Resistor_SMD:R_0402_1005Metric, symbol Device:R_Small
- added R8: 1K, Resistor_SMD:R_0402_1005Metric, symbol Device:R_Small
- added R9: 100K, Resistor_SMD:R_0402_1005Metric, symbol Device:R_Small
- added U4: MCP73831, Package_TO_SOT_SMD:SOT-23-5, symbol Battery_Management_Extra:MCP73831
Connections:
- net GND: now also C16.1, C18.2, C9.2, J1.2 (Pin_2), J3.2 (Pin_2), R7.1, R9.1, U4.2 (GND)
- net VCC: now also J2.4 (Pin_4), C9.1, D5.1 (K), Q1.2 (S)
- new net: D4.1 (K), R8.1
- new net: R8.2, U4.1 (STAT)
- new net: R7.2, U4.5 (PROG)
- new net VBAT: C16.2, J3.1 (Pin_1), Q1.3 (D), U4.3 (VBAT)
- new net VIN: C18.1, D4.2 (A), D5.2 (A), J1.1 (Pin_1), Q1.1 (G), R9.2, U4.4 (VDD)

Commit message: V2
Parts:
- removed C5: 68pF, Capacitor_SMD:C_0603_1608Metric, symbol Device:C_Small
- removed C6: 330pF, Capacitor_SMD:C_0603_1608Metric, symbol Device:C_Small
- removed C7: as large as possible, Capacitor_Tantalum_SMD:CP_EIA-3528-12_Kemet-T, symbol Device:C_Polarized_Small
- removed C8: 4,7µF, Capacitor_SMD:C_0603_1608Metric, symbol Device:C_Small
- removed D2: D, Diode_SMD:D_SOD-323, symbol Device:D_Small
- removed D4: LED_CHR, LED_SMD:LED_0402_1005Metric, symbol Device:LED_Small
- removed D5: D_Schottky_Small, Diode_SMD:D_SOD-323, symbol Device:D_Schottky_Small
- removed J1: Conn_01x02, symbol Connector_Generic:Conn_01x02
- removed L1, L2: 4,7µH, Inductor_SMD:L_0805_2012Metric, symbol Device:L_Small
- removed R2: 42k, Resistor_SMD:R_0603_1608Metric, symbol Device:R_Small
- removed U1: R1283K001C-TR, footprints:PE-DFNPL2730-12-180404_NMD, symbol 2025-10-09_16-12-42:R1283K001C-TR
- added C11, C12, C14: 10µF, Capacitor_SMD:C_0603_1608Metric, symbol Device:C_Small
- added C13, C15: 1µF, Capacitor_SMD:C_0603_1608Metric, symbol Device:C_Small
- added D2: LED_CHR, LED_THT:LED_D3.0mm, symbol Device:LED_Small
- added D3, D4, D5, D6: D, Diode_SMD:D_SOD-323, symbol Device:D_Small
- added D7: 18V, Diode_SMD:D_SOD-323, symbol Device:D_Zener_Small
- added F1: Fuse, Fuse:Fuse_1206_3216Metric, symbol Device:Fuse_Small
- added J4: Conn_01x01, Connector_PinHeader_2.54mm:PinHeader_1x01_P2.54mm_Vertical, symbol Connector_Generic:Conn_01x01
- added JP1: Jumper, Jumper:SolderJumper-2_P1.3mm_Open_RoundedPad1.0x1.5mm, symbol Jumper:Jumper_2_Small_Open
- added L3, L4, L5: 10µH, Inductor_SMD:L_APV_ANR5040, symbol Device:L_Small
- added R10, R11: 100k, Resistor_SMD:R_0603_1608Metric, symbol Device:R_Small
- added R12: 6,8k, Resistor_SMD:R_0603_1608Metric, symbol Device:R_Small
- added R13: 15k, Resistor_SMD:R_0603_1608Metric, symbol Device:R_Small
- added R14: TBD, Resistor_SMD:R_0603_1608Metric, symbol Device:R_Small
- added U2, U3: LGS6302B5, Package_TO_SOT_SMD:SOT-23-5, symbol Regulator_Switching:LGS6302B5
- C1: value 4,7µF -> 10µF
- C18: footprint Capacitor_SMD:C_0402_1005Metric -> Capacitor_SMD:C_0603_1608Metric
- C3: footprint Capacitor_SMD:C_0603_1608Metric -> Capacitor_SMD:C_1206_3216Metric
- C4: value 100nF -> 10µF
- C9: value TBD -> 1µF; footprint Capacitor_SMD:C_0402_1005Metric -> Capacitor_SMD:C_0603_1608Metric
- J3: footprint (none) -> Connector_JST:JST_PH_S2B-PH-K_1x02_P2.00mm_Horizontal
- R1: value 10k -> 33k
- R3: value 1k -> 100k
- R4: value 6,8k -> 1K
- R5: value 100k -> 100K
- R6: value 1k -> 2K
- R7: value 2K -> 100k; footprint Resistor_SMD:R_0402_1005Metric -> Resistor_SMD:R_0603_1608Metric
- R8: value 1K -> 100k; footprint Resistor_SMD:R_0402_1005Metric -> Resistor_SMD:R_0603_1608Metric
- R9: value 100K -> 100k; footprint Resistor_SMD:R_0402_1005Metric -> Resistor_SMD:R_0603_1608Metric
Connections:
- net +5V: now also C4.1, R7.1; no longer R3.1
- net GND: now also J3.1 (Pin_1), R3.2, R5.1, R6.1, C11.2, C12.2, C14.2, C15.2, D6.1 (K), D7.1 (K), L4.2, R10.2, R12.2, R13.2, U2.2 (GND), U3.2 (GND); no longer C9.2, J3.2 (Pin_2), R7.1, R9.1
- net VBAT: now also J3.2 (Pin_2); no longer J3.1 (Pin_1)
- net VCC: now also R8.2, R9.2, C11.1, C12.1, D3.1 (K), F1.2, JP1.2 (B), L3.1, L5.1, U2.5 (IN), U3.5 (IN); no longer C9.1, J2.4 (Pin_4)
- net VIN: now also R5.2, D2.2 (A), D3.2 (A), J4.1 (Pin_1), JP1.1 (A); no longer R9.2
- net at R8.1: now also R3.1, U3.4 (EN)
- net at U4.1 (STAT): now also R4.2; no longer R8.2
- net at U4.5 (PROG): now also R6.2; no longer R7.2
- net -VDC renamed -18V
- net -18V: now also D7.2 (A), R14.2; no longer R5.1, R6.1
- net FB1: no longer names the net of R1.1
- net FB1: now also R7.2, U3.3 (FB)
- net FB2: no longer names the net of R4.1
- net FB2: now also D2.1 (K); no longer R5.2
- removed net VREF: C4.1, R4.2
- net buck+ renamed sw2
- net sw2: now also C9.2, L4.1
- new net: F1.1, J2.4 (Pin_4)
- new net: R11.2, R12.1, U2.3 (FB)
- new net: R10.1, R9.1, U2.4 (EN)
- new net +18V: C14.1, D4.1 (K), R11.1
- new net pump1: C13.2, D5.1 (K), D6.2 (A)
- new net pump2: C15.1, D5.2 (A), R13.1, R14.1
- new net sw: C9.1, L3.2, U3.1 (SW)
- new net sw3: C13.1, D4.2 (A), L5.2, U2.1 (SW)
- no-connect marks 1 -> 0
Other:
- moved on the sheet: C10, C16, C18, C2, C3, D1, J2, J3, Q1, R1, R3, U4

Commit message: some things i missed
Parts:
- removed F1: Fuse, Fuse:Fuse_1206_3216Metric, symbol Device:Fuse_Small
- added J1: Conn_01x01, Connector_PinHeader_2.54mm:PinHeader_1x01_P2.54mm_Vertical, symbol Connector_Generic:Conn_01x01
- added JP2: Jumper, Jumper:SolderJumper-2_P1.3mm_Open_RoundedPad1.0x1.5mm, symbol Jumper:Jumper_2_Small_Open
- added RV1: Varistor, Resistor_SMD:R_0603_1608Metric, symbol Device:Varistor
- C1, C11, C12, C14, C16, C2, C4: footprint Capacitor_SMD:C_0603_1608Metric -> Capacitor_SMD:C_0805_2012Metric
- C10: footprint Capacitor_Tantalum_SMD:CP_EIA-3528-12_Kemet-T -> Capacitor_SMD:C_1206_3216Metric
- C3: footprint Capacitor_SMD:C_1206_3216Metric -> Capacitor_SMD:C_0805_2012Metric
- JP1: now left out of the parts list
Connections:
- net GND: now also J3.2 (Pin_2), RV1.2; no longer J3.1 (Pin_1)
- net VBAT: now also J3.1 (Pin_1); no longer J3.2 (Pin_2)
- net VCC: now also J2.4 (Pin_4), JP2.2 (B); no longer D3.1 (K), Q1.2 (S)
- net VIN: now also RV1.1
- new net: D3.1 (K), J1.1 (Pin_1), JP2.1 (A), Q1.2 (S)

Commit message: final tweaks before manufacture
Parts:
- added C5: 1µF, Capacitor_SMD:C_0603_1608Metric, symbol Device:C_Small
- C10: value as large as possible -> 100µF
- C3: value 10µF -> 100µF; footprint Capacitor_SMD:C_0805_2012Metric -> Capacitor_SMD:C_1206_3216Metric
Connections:
- net -18V: now also C5.1
- net GND: now also C5.2
Other:
- moved on the sheet: D7
Changed lines of the file:
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@@
 	)
 	(junction
+		(at 95.25 90.17)
+		(diameter 0)
+		(color 0 0 0 0)
+	)
+	(junction
 		(at 68.58 121.92)
 		(diameter 0)
@@
 	)
 	(junction
-		(at 96.52 90.17)
+		(at 99.06 90.17)
 		(diameter 0)
 		(color 0 0 0 0)
@@
 	)
 	(junction
-		(at 96.52 82.55)
+		(at 99.06 82.55)
 		(diameter 0)
 		(color 0 0 0 0)
@@
 	)
 	(junction
+		(at 95.25 82.55)
+		(diameter 0)
+		(color 0 0 0 0)
+	)
+	(junction
 		(at 82.55 82.55)
 		(diameter 0)
@@
 	(wire
 		(pts
-			(xy 96.52 90.17) (xy 96.52 91.44)
+			(xy 99.06 90.17) (xy 99.06 91.44)
 		)
 		(stroke
@@
 	(wire
 		(pts
-			(xy 93.98 82.55) (xy 96.52 82.55)
+			(xy 99.06 82.55) (xy 99.06 83.82)
 		)
 		(stroke
@@
 	(wire
 		(pts
-			(xy 96.52 82.55) (xy 96.52 83.82)
+			(xy 25.4 45.72) (xy 25.4 46.99)
 		)
 		(stroke
@@
 	(wire
 		(pts
-			(xy 25.4 45.72) (xy 25.4 46.99)
+			(xy 66.04 97.79) (xy 67.31 97.79)
 		)
 		(stroke
@@
 	(wire
 		(pts
-			(xy 66.04 97.79) (xy 67.31 97.79)
+			(xy 64.77 62.23) (xy 64.77 63.5)
 		)
 		(stroke
 			(width 0)
-			(type default)
+			(type solid)
 		)
 	)
 	(wire
 		(pts
-			(xy 64.77 62.23) (xy 64.77 63.5)
+			(xy 48.26 29.21) (xy 48.26 35.56)
 		)
 		(stroke
@@
 	(wire
 		(pts
-			(xy 48.26 29.21) (xy 48.26 35.56)
+			(xy 95.25 90.17) (xy 99.06 90.17)
 		)
 		(stroke
 			(width 0)
-			(type solid)
+			(type default)
 		)
 	)
@@
 	(wire
 		(pts
-			(xy 82.55 29.21) (xy 82.55 27.94)
+			(xy 95.25 88.9) (xy 95.25 90.17)
 		)
 		(stroke
@@
 	(wire
 		(pts
-			(xy 68.58 101.6) (xy 74.93 101.6)
+			(xy 82.55 29.21) (xy 82.55 27.94)
 		)
 		(stroke
@@
 	(wire
 		(pts
-			(xy 86.36 90.17) (xy 96.52 90.17)
+			(xy 68.58 101.6) (xy 74.93 101.6)
 		)
 		(stroke
@@
 	(wire
 		(pts
+			(xy 95.25 82.55) (xy 95.25 83.82)
+		)
+		(stroke
+			(width 0)
+			(type default)
+		)
+	)
+	(wire
+		(pts
 			(xy 57.15 97.79) (xy 66.04 97.79)
 		)
@@
 	(wire
 		(pts
+			(xy 93.98 82.55) (xy 95.25 82.55)
+		)
+		(stroke
+			(width 0)
+			(type default)
+		)
+	)
+	(wire
+		(pts
 			(xy 99.06 27.94) (xy 107.95 27.94)
 		)
@@
 	(wire
 		(pts
-			(xy 96.52 81.28) (xy 96.52 82.55)
+			(xy 99.06 81.28) (xy 99.06 82.55)
 		)
 		(stroke
@@
 	(wire
 		(pts
+			(xy 86.36 90.17) (xy 95.25 90.17)
+		)
+		(stroke
+			(width 0)
+			(type default)
+		)
+	)
+	(wire
+		(pts
 			(xy 74.93 96.52) (xy 74.93 97.79)
 		)
@@
 	(wire
 		(pts
-			(xy 96.52 88.9) (xy 96.52 90.17)
+			(xy 99.06 88.9) (xy 99.06 90.17)
 		)
 		(stroke
@@
 	(wire
 		(pts
+			(xy 95.25 82.55) (xy 99.06 82.55)
+		)
+		(stroke
+			(width 0)
+			(type default)
+		)
+	)
+	(wire
+		(pts
 			(xy 31.75 121.92) (xy 40.64 121.92)
 		)
@@
 	)
 	(symbol
+		(lib_id "Device:C_Small")
+		(at 95.25 86.36 0)
+		(unit 1)
+		(exclude_from_sim no)
+		(in_bom yes)
+		(on_board yes)
+		(dnp no)
+		(property "Reference" "C5"
+			(at 97.282 94.488 0)
+			(effects
+				(font
+					(size 1.27 1.27)
+				)
+				(justify right)
+			)
+		)
+		(property "Value" "1µF"
+			(at 97.282 91.948 0)
+			(effects
+				(font
+					(size 1.27 1.27)
+				)
+				(justify right)
+			)
+		)
+		(property "Footprint" "Capacitor_SMD:C_0603_1608Metric"
+			(at 95.25 86.36 0)
+			(effects
+				(font
+					(size 1.27 1.27)
+				)
+				(hide yes)
+			)
+		)
+		(property "Datasheet" "~"
+			(at 95.25 86.36 0)
+			(effects
+				(font
+					(size 1.27 1.27)
+				)
+				(hide yes)
+			)
+		)
+		(property "Description" "Unpolarized capacitor, small symbol"
+			(at 95.25 86.36 0)
+			(effects
+				(font
+					(size 1.27 1.27)
+				)
+				(hide yes)
+			)
+		)
+		(pin "1"
+		)
+		(pin "2"
+		)
+		(instances
+			(project "GB_DMG_PSU"
+				(path "/3b465854-de6d-4c79-a332-83f1753a534a"
+					(reference "C5")
+					(unit 1)
+				)
+			)
+		)
+	)
+	(symbol
 		(lib_id "Device:D_Small")
 		(at 135.89 27.94 180)
@@
 	(symbol
 		(lib_id "Device:D_Zener_Small")
-		(at 96.52 86.36 90)
+		(at 99.06 86.36 90)
 		(unit 1)
 		(exclude_from_sim no)
@@
 		(fields_autoplaced yes)
 		(property "Reference" "D7"
-			(at 99.06 85.0899 90)
+			(at 101.6 85.0899 90)
 			(effects
 				(font
@@
 		)
 		(property "Value" "18V"
-			(at 99.06 87.6299 90)
+			(at 101.6 87.6299 90)
 			(effects
 				(font
@@
 		)
 		(property "Footprint" "Diode_SMD:D_SOD-323"
-			(at 96.52 86.36 90)
+			(at 99.06 86.36 90)
 			(effects
 				(font
@@
 		)
 		(property "Datasheet" "~"
-			(at 96.52 86.36 90)
+			(at 99.06 86.36 90)
 			(effects
 				(font
@@
 		)
 		(property "Description" "Zener diode, small symbol"
-			(at 96.52 86.36 0)
+			(at 99.06 86.36 0)
 			(effects
 				(font
@@
 	(symbol
 		(lib_id "power:-15V")
-		(at 96.52 81.28 0)
+		(at 99.06 81.28 0)
 		(unit 1)
 		(exclude_from_sim no)
@@
 		(dnp no)
 		(property "Reference" "#PWR02"
-			(at 96.52 85.09 0)
+			(at 99.06 85.09 0)
 			(effects
 				(font
@@
 		)
 		(property "Value" "-18V"
-			(at 96.52 77.47 0)
+			(at 99.06 77.47 0)
 			(effects
 				(font
@@
 		)
 		(property "Footprint" ""
-			(at 96.52 81.28 0)
+			(at 99.06 81.28 0)
 			(effects
 				(font
@@
 		)
 		(property "Datasheet" ""
-			(at 96.52 81.28 0)
+			(at 99.06 81.28 0)
 			(effects
 				(font
@@
 		)
 		(property "Description" "Power symbol creates a global label with name \"-15V\""
-			(at 96.52 81.28 0)
+			(at 99.06 81.28 0)
 			(effects
 				(font
@@
 			)
 		)
-		(property "Value" "10µF"
+		(property "Value" "100µF"
 			(at 156.718 57.404 0)
 			(effects
@@
 			)
 		)
-		(property "Footprint" "Capacitor_SMD:C_0805_2012Metric"
+		(property "Footprint" "Capacitor_SMD:C_1206_3216Metric"
 			(at 163.83 55.88 0)
 			(effects
@@
 			)
 		)
-		(property "Value" "as large as possible"
+		(property "Value" "100µF"
 			(at 164.846 22.6442 0)
 			(effects
@@
 		(lib_name "GND_1")
 		(lib_id "power:GND")
-		(at 96.52 91.44 0)
+		(at 99.06 91.44 0)
 		(unit 1)
 		(exclude_from_sim no)
@@
 		(dnp no)
 		(property "Reference" "#PWR028"
-			(at 96.52 97.79 0)
+			(at 99.06 97.79 0)
 			(effects
 				(font
@@
 		)
 		(property "Value" "GND"
-			(at 96.52 95.504 0)
+			(at 99.06 95.504 0)
 			(effects
 				(font
@@
 		)
 		(property "Footprint" ""
-			(at 96.52 91.44 0)
+			(at 99.06 91.44 0)
 			(effects
 				(font
@@
 		)
 		(property "Datasheet" ""
-			(at 96.52 91.44 0)
+			(at 99.06 91.44 0)
 			(effects
 				(font
@@
 		)
 		(property "Description" "Power symbol creates a global label with name \"GND\" , ground"
-			(at 96.52 91.44 0)
+			(at 99.06 91.44 0)
 			(effects
 				(font
