File: GB_DMG_PSU.kicad_sch (KiCad schematic)
At the start: 32 parts, among them J2 Conn_01x04, U2 LGS6302B5, U3 LGS6302B5

Commit message: BOM/gerbers
Parts:
- C3: value 100µF -> 22µF
Changed lines of the file:
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@@
 			)
 		)
-		(property "Value" "100µF"
+		(property "Value" "22µF"
 			(at 156.718 57.404 0)
 			(effects
